Commit message: Changed urdf to align with the proper axes

File: pupper_description/pupper.urdf (robot description, URDF)
Before this commit: robot pupper, 41 links, 40 joints
Links:
- link back_left_cover: geometry 
- link back_left_elbow: geometry 
- link back_left_foot: geometry 
- link back_left_hip: geometry 
- link back_left_hub: geometry 
- link back_left_lower_link: geometry 
- link back_left_shoulder: geometry 
- link back_left_shroud: geometry 
- link back_left_upper_link: geometry 
- link back_right_cover: geometry 
- link back_right_elbow: geometry 
- link back_right_foot: geometry 
- link back_right_hip: geometry 
- link back_right_hub: geometry 
- link back_right_lower_link: geometry 
- link back_right_shoulder: geometry 
- link back_right_shroud: geometry 
- link back_right_upper_link: geometry 
- link battery: geometry 
- link bottom_PCB: geometry 
- link front_bulkhead: geometry 
- link front_left_cover: geometry 
- link front_left_elbow: geometry 
- link front_left_foot: geometry 
- link front_left_hip: geometry 
- link front_left_hub: geometry 
- link front_left_lower_link: geometry 
- link front_left_shoulder: geometry 
- link front_left_upper_link: geometry 
- link front_right_cover: geometry 
- link front_right_elbow: geometry 
- link front_right_foot: geometry 
- link front_right_hip: geometry 
- link front_right_hub: geometry 
- link front_right_lower_link: geometry 
- link front_right_shoulder: geometry 
- link front_right_upper_link: geometry 
- link middle_bulkhead_front: geometry 
- link middle_bulkhead_rear: geometry 
- link rear_bulkhead: geometry 
- link top_PCB: geometry 
Joints:
- joint back_left_hip_fixed_joint: origin xyz=0.05 0.095 0.044 rpy=-1.5707963268 0 0 -> xyz=-0.097 0.0425 0.041 rpy=-1.5707963268 0 1.5707963268
- joint back_left_shroud_to_base: origin xyz=0.003 0.113 0.044 rpy=1.5707963268 3.14159265359 0 -> xyz=-0.114 -0.004 0.044 rpy=1.5707963268 0 1.5707963268
- joint back_right_hip_fixed_joint: origin xyz=-0.045 0.095 0.044 rpy=-1.5707963268 0 0 -> xyz=-0.097 -0.0505 0.041 rpy=-1.5707963268 0 1.5707963268
- joint battery_to_body: origin xyz=0.002 0.03 0.02425 -> xyz=-0.015 -0.004 0.02425 rpy=0 0 1.5707963268
- joint front_bulkhead_to_base: origin xyz=0.002 0.114 0.044 rpy=1.5707963268 0 0 -> xyz=-0.114 -0.004 0.044 rpy=1.5707963268 0 1.5707963268
- joint front_left_hip_fixed_joint: origin xyz=0.05 -0.105 0.044 rpy=-1.5707963268 0 0 -> xyz=0.104 0.0425 0.041 rpy=-1.5707963268 0 1.5707963268
- joint front_right_hip_fixed_joint: origin xyz=-0.045 -0.105 0.044 rpy=-1.5707963268 0 0 -> xyz=0.104 -0.0505 0.041 rpy=-1.5707963268 0 1.5707963268
- joint middle_bulkhead_to_base_1: origin xyz=0.002 0.114 0.044 rpy=1.5707963268 0 0 -> xyz=-0.114 -0.004 0.044 rpy=1.5707963268 0 1.5707963268
- joint middle_bulkhead_to_base_2: origin xyz=0.003 0.114 0.044 rpy=1.5707963268 0 0 -> xyz=-0.114 -0.004 0.044 rpy=1.5707963268 0 1.5707963268
- joint rear_bulk_head_to_body: origin xyz=0.003 0.113 0.044 rpy=1.5707963268 0 0 -> xyz=-0.114 -0.004 0.044 rpy=1.5707963268 0 1.5707963268
- joint right_shroud_to_base: origin xyz=0.003 0.113 0.044 rpy=1.5707963268 3.14159265359 0 -> xyz=-0.114 -0.004 0.044 rpy=1.5707963268 0 1.5707963268
- joint top_PCB_to_base: origin xyz=0 0 0.088 rpy=0 0 0 -> xyz=0 -0.0075 0.088 rpy=0 0 1.5707963268

File: pupper_description/pupper.urdf.xacro (robot description, xacro)
@@ -52,10 +52,10 @@
         <visual name = "bottom_PCB_visual">
             <geometry>
-                <mesh filename = "${VisualPath}/Body/PCB_Board_Shifted.dae" scale = "${meshScale_in}"/>
+                <mesh filename = "${VisualPath}/Body/PCB_Board.stl" scale = "${meshScale_in}"/>
             </geometry>
         </visual>
         <collision name = "bottom_PCB_collision">
             <geometry>
-                <mesh filename = "${CollisionPath}/Body/PCB_Board_Shifted.dae" scale = "${meshScale_in}"/>
+                <mesh filename = "${CollisionPath}/Body/PCB_Board.stl" scale = "${meshScale_in}"/>
             </geometry>
         </collision>
@@ -86,5 +86,5 @@
         <parent link = "bottom_PCB"/>
         <child  link = "front_bulkhead"/>
-        <origin xyz = "0.002 0.114 0.044" rpy = "${PI/2} 0 0"/>
+        <origin xyz = "-0.114 -0.004 0.044" rpy = "${PI/2} 0 ${PI/2}"/>
     </joint>
     <!-- Create Middle Bulkhead -->
@@ -112,5 +112,5 @@
         <parent link = "bottom_PCB"/>
         <child  link = "middle_bulkhead_front"/>
-        <origin xyz = "0.002 0.114 0.044" rpy = "${PI/2} 0 0"/>
+        <origin xyz = "-0.114 -0.004 0.044" rpy = "${PI/2} 0 ${PI/2}"/>
     </joint>
     <!-- Create 2nd Middle Bulkhead -->
@@ -138,5 +138,5 @@
         <parent link = "bottom_PCB"/>
         <child  link = "middle_bulkhead_rear"/>
-        <origin xyz = "0.003 0.114 0.044" rpy = "${PI/2} 0 0"/>
+        <origin xyz = "-0.114 -0.004 0.044" rpy = "${PI/2} 0 ${PI/2}"/>
     </joint>
     <!-- Create back right shroud -->
@@ -164,5 +164,5 @@
         <parent link = "bottom_PCB"/>
         <child  link = "back_right_shroud"/>
-        <origin xyz  = "0.003 0.113 0.044" rpy = "${PI/2} ${PI} 0"/>
+        <origin xyz  = "-0.114 -0.004 0.044" rpy = "${PI/2} 0 ${PI/2}"/>
     </joint>
     <!-- Create back left shroud -->
@@ -191,5 +191,5 @@
         <parent link = "bottom_PCB"/>
         <child  link = "back_left_shroud"/>
-        <origin xyz  = "0.003 0.113 0.044" rpy = "${PI/2} ${PI} 0"/>
+        <origin xyz = "-0.114 -0.004 0.044" rpy = "${PI/2} 0 ${PI/2}"/>
     </joint>
     <!-- Create rear bulkhead -->
@@ -217,5 +217,5 @@
         <parent link = "bottom_PCB"/>
         <child  link = "rear_bulkhead"/>
-        <origin xyz = "0.003 0.113 0.044" rpy = "${PI/2} 0 0"/>
+        <origin xyz = "-0.114 -0.004 0.044" rpy = "${PI/2} 0 ${PI/2}"/>
     </joint>
     <!-- Create a bulk mass for the battery -->
@@ -244,5 +244,5 @@
         <parent link = "bottom_PCB"/>
         <child  link = "battery"/>
-        <origin xyz = "0.002 0.03 ${batt_z/2}"/>
+        <origin xyz = "-0.015 -0.004 ${batt_z/2}" rpy = "0 0 ${PI/2}"/>
     </joint>
     <!-- Create top plate -->
@@ -269,17 +269,17 @@
         <parent link = "bottom_PCB"/>
         <child  link = "top_PCB"/>
-        <origin xyz  = "0 0 0.088" rpy = "0 0 0"/>
+        <origin xyz  = "0 -0.0075 0.088" rpy = "0 0 ${PI/2}"/>
     </joint>
     <xacro:leftLeg name = "front" parent = "bottom_PCB">
-        <origin xyz = "0.05 -0.105 0.044" rpy = "${-PI/2} 0 0"/>
+        <origin xyz = "0.104 0.0425 0.041" rpy = "${-PI/2} 0 ${PI/2}"/>
     </xacro:leftLeg>
     <xacro:leftLeg name = "back" parent = "bottom_PCB">
-        <origin xyz = "0.05 0.095 0.044" rpy = "${-PI/2} 0 0"/>
+        <origin xyz = "-0.097 0.0425 0.041" rpy = "${-PI/2} 0 ${PI/2}"/>
     </xacro:leftLeg>
     <xacro:rightLeg name = "front" parent = "bottom_PCB">
-        <origin xyz = "-0.045 -0.105 0.044" rpy = "${-PI/2} 0 0"/>
+        <origin xyz = "0.104 -0.0505 0.041" rpy = "${-PI/2} 0 ${PI/2}"/>
     </xacro:rightLeg>
     <xacro:rightLeg name = "back" parent = "bottom_PCB">
-        <origin xyz = "-0.045 0.095 0.044" rpy = "${-PI/2} 0 0"/>
+        <origin xyz = "-0.097 -0.0505 0.041" rpy = "${-PI/2} 0 ${PI/2}"/>
     </xacro:rightLeg>
 </robot>

Commit message: Many changes

File: pupper_description/pupper.urdf (robot description, URDF)
Before this commit: robot pupper, 41 links, 40 joints
Joints:
- joint back_left_hip_fixed_joint: origin xyz=-0.097 0.0425 0.041 rpy=-1.5707963268 0 1.5707963268 -> xyz=-0.11 0.045 0.041 rpy=4.71238898039 0 1.5707963268
- joint back_left_shroud_to_base: origin xyz=-0.114 -0.004 0.044 rpy=1.5707963268 0 1.5707963268 -> xyz=-0.128 0.00 0.044 rpy=1.5707963268 0 1.5707963268
- joint back_right_hip_fixed_joint: origin xyz=-0.097 -0.0505 0.041 rpy=-1.5707963268 0 1.5707963268 -> xyz=-0.11 -0.045 0.041 rpy=4.71238898039 0 1.5707963268
- joint battery_to_body: origin xyz=-0.015 -0.004 0.02425 rpy=0 0 1.5707963268 -> xyz=-0.028 0.00 0.02425 rpy=0 0 1.5707963268
- joint front_bulkhead_to_base: origin xyz=-0.114 -0.004 0.044 rpy=1.5707963268 0 1.5707963268 -> xyz=-0.128 0.00 0.044 rpy=1.5707963268 0 1.5707963268
- joint front_left_hip_fixed_joint: origin xyz=0.104 0.0425 0.041 rpy=-1.5707963268 0 1.5707963268 -> xyz=0.091 0.045 0.041 rpy=4.71238898039 0 1.5707963268
- joint front_right_hip_fixed_joint: origin xyz=0.104 -0.0505 0.041 rpy=-1.5707963268 0 1.5707963268 -> xyz=0.091 -0.045 0.041 rpy=4.71238898039 0 1.5707963268
- joint middle_bulkhead_to_base_1: origin xyz=-0.114 -0.004 0.044 rpy=1.5707963268 0 1.5707963268 -> xyz=-0.128 0.00 0.044 rpy=1.5707963268 0 1.5707963268
- joint middle_bulkhead_to_base_2: origin xyz=-0.114 -0.004 0.044 rpy=1.5707963268 0 1.5707963268 -> xyz=-0.128 0.00 0.044 rpy=1.5707963268 0 1.5707963268
- joint rear_bulk_head_to_body: origin xyz=-0.114 -0.004 0.044 rpy=1.5707963268 0 1.5707963268 -> xyz=-0.128 0.00 0.044 rpy=1.5707963268 0 1.5707963268
- joint right_shroud_to_base: origin xyz=-0.114 -0.004 0.044 rpy=1.5707963268 0 1.5707963268 -> xyz=-0.128 0.00 0.044 rpy=1.5707963268 0 1.5707963268
- joint top_PCB_to_base: origin xyz=0 -0.0075 0.088 rpy=0 0 1.5707963268 -> xyz=0.00 0.00 0.087 rpy=0 0 0

File: pupper_description/pupper.urdf.xacro (robot description, xacro)
@@ -86,5 +86,5 @@
         <parent link = "bottom_PCB"/>
         <child  link = "front_bulkhead"/>
-        <origin xyz = "-0.114 -0.004 0.044" rpy = "${PI/2} 0 ${PI/2}"/>
+        <origin xyz = "-0.128 0.00 0.044" rpy = "${PI/2} 0 ${PI/2}"/>
     </joint>
     <!-- Create Middle Bulkhead -->
@@ -112,5 +112,5 @@
         <parent link = "bottom_PCB"/>
         <child  link = "middle_bulkhead_front"/>
-        <origin xyz = "-0.114 -0.004 0.044" rpy = "${PI/2} 0 ${PI/2}"/>
+        <origin xyz = "-0.128 0.00 0.044" rpy = "${PI/2} 0 ${PI/2}"/>
     </joint>
     <!-- Create 2nd Middle Bulkhead -->
@@ -138,5 +138,5 @@
         <parent link = "bottom_PCB"/>
         <child  link = "middle_bulkhead_rear"/>
-        <origin xyz = "-0.114 -0.004 0.044" rpy = "${PI/2} 0 ${PI/2}"/>
+        <origin xyz = "-0.128 0.00 0.044" rpy = "${PI/2} 0 ${PI/2}"/>
     </joint>
     <!-- Create back right shroud -->
@@ -164,5 +164,5 @@
         <parent link = "bottom_PCB"/>
         <child  link = "back_right_shroud"/>
-        <origin xyz  = "-0.114 -0.004 0.044" rpy = "${PI/2} 0 ${PI/2}"/>
+        <origin xyz = "-0.128 0.00 0.044" rpy = "${PI/2} 0 ${PI/2}"/>
     </joint>
     <!-- Create back left shroud -->
@@ -191,5 +191,5 @@
         <parent link = "bottom_PCB"/>
         <child  link = "back_left_shroud"/>
-        <origin xyz = "-0.114 -0.004 0.044" rpy = "${PI/2} 0 ${PI/2}"/>
+        <origin xyz = "-0.128 0.00 0.044" rpy = "${PI/2} 0 ${PI/2}"/>
     </joint>
     <!-- Create rear bulkhead -->
@@ -217,5 +217,5 @@
         <parent link = "bottom_PCB"/>
         <child  link = "rear_bulkhead"/>
-        <origin xyz = "-0.114 -0.004 0.044" rpy = "${PI/2} 0 ${PI/2}"/>
+        <origin xyz = "-0.128 0.00 0.044" rpy = "${PI/2} 0 ${PI/2}"/>
     </joint>
     <!-- Create a bulk mass for the battery -->
@@ -244,5 +244,5 @@
         <parent link = "bottom_PCB"/>
         <child  link = "battery"/>
-        <origin xyz = "-0.015 -0.004 ${batt_z/2}" rpy = "0 0 ${PI/2}"/>
+        <origin xyz = "-0.028 0.00 ${batt_z/2}" rpy = "0 0 ${PI/2}"/>
     </joint>
     <!-- Create top plate -->
@@ -255,10 +255,10 @@
         <visual name = "top_PCB_visual">
             <geometry>
-                <mesh filename = "${VisualPath}/Body/PCB_Board_Shifted.dae" scale = "${meshScale_in}"/>
+                <mesh filename = "${VisualPath}/Body/PCB_Board.stl" scale = "${meshScale_in}"/>
             </geometry>
         </visual>
         <collision name = "top_PCB_collision">
             <geometry>
-                <mesh filename = "${CollisionPath}/Body/PCB_Board_Shifted.dae" scale = "${meshScale_in}"/>
+                <mesh filename = "${CollisionPath}/Body/PCB_Board.stl" scale = "${meshScale_in}"/>
             </geometry>
         </collision>
@@ -269,17 +269,17 @@
         <parent link = "bottom_PCB"/>
         <child  link = "top_PCB"/>
-        <origin xyz  = "0 -0.0075 0.088" rpy = "0 0 ${PI/2}"/>
+        <origin xyz  = "0.00 0.00 0.087" rpy = "0 0 0"/>
     </joint>
     <xacro:leftLeg name = "front" parent = "bottom_PCB">
-        <origin xyz = "0.104 0.0425 0.041" rpy = "${-PI/2} 0 ${PI/2}"/>
+        <origin xyz = "0.091 0.045 0.041" rpy = "${3*PI/2} 0 ${PI/2}"/>
     </xacro:leftLeg>
     <xacro:leftLeg name = "back" parent = "bottom_PCB">
-        <origin xyz = "-0.097 0.0425 0.041" rpy = "${-PI/2} 0 ${PI/2}"/>
+        <origin xyz = "-0.11 0.045 0.041" rpy = "${3*PI/2} 0 ${PI/2}"/>
     </xacro:leftLeg>
     <xacro:rightLeg name = "front" parent = "bottom_PCB">
-        <origin xyz = "0.104 -0.0505 0.041" rpy = "${-PI/2} 0 ${PI/2}"/>
+        <origin xyz = "0.091 -0.045 0.041" rpy = "${3*PI/2} 0 ${PI/2}"/>
     </xacro:rightLeg>
     <xacro:rightLeg name = "back" parent = "bottom_PCB">
-        <origin xyz = "-0.097 -0.0505 0.041" rpy = "${-PI/2} 0 ${PI/2}"/>
+        <origin xyz = "-0.11 -0.045 0.041" rpy = "${3*PI/2} 0 ${PI/2}"/>
     </xacro:rightLeg>
 </robot>
