Commit message: Made joint names more uniform

File: pupper_description/left_leg.xacro (robot description, xacro)
@@ -41,9 +41,4 @@
             </collision>
         </link>
-        <!-- Join the Hub and the Upper Link with a motor -->
-        <xacro:motor name = "${name}_left_shoulder" axis = "1 0 0" fixed_parent = "${hubName}" revolute_child = "${upperName}">
-            <origin xyz = "0 0 0.005" rpy = "0 0 0"/>
-            <origin xyz = "0 0 0.022" rpy = "0 ${-PI/2} 0"/>
-        </xacro:motor>
         <!-- Create the covering for the upper portion of the leg -->
         <xacro:property name = "upperCoverName" value = "${name}_left_leg_cover"/>
@@ -90,4 +85,14 @@
             </collision>
         </link>
+        <!-- Connect leg to parent with a motor -->
+        <xacro:motor name = "${name}_left_shoulder_1" axis = "-1 0 0" fixed_parent = "${parent}" revolute_child = "${hubName}">
+            <xacro:insert_block name = "origin"/>
+            <origin xyz = "0 0 0.036" rpy = "0 ${PI/2} 0"/>
+        </xacro:motor>
+        <!-- Join the Hub and the Upper Link with a motor -->
+        <xacro:motor name = "${name}_left_shoulder_2" axis = "1 0 0" fixed_parent = "${hubName}" revolute_child = "${upperName}">
+            <origin xyz = "0 0 0.005" rpy = "0 0 0"/>
+            <origin xyz = "0 0 0.022" rpy = "0 ${-PI/2} 0"/>
+        </xacro:motor>
         <!-- Connect Upper Link and Lower Link with a motor -->
         <xacro:motor name = "${name}_left_elbow" axis = "0 0 -1" fixed_parent = "${upperName}" revolute_child = "${lowerName}">
@@ -95,9 +100,4 @@
             <origin xyz = "0 0 -0.032" rpy = "${PI} ${PI} 0"/>
         </xacro:motor>
-        <!-- Connect leg to parent with a motor -->
-        <xacro:motor name = "${name}_left_parent_motor" axis = "-1 0 0" fixed_parent = "${parent}" revolute_child = "${hubName}">
-            <xacro:insert_block name = "origin"/>
-            <origin xyz = "0 0 0.036" rpy = "0 ${PI/2} 0"/>
-        </xacro:motor>
     </xacro:macro>
 </robot>

File: pupper_description/right_leg.xacro (robot description, xacro)
@@ -41,9 +41,4 @@
             </collision>
         </link>
-        <!-- Join the Hub and the Upper Link with a motor -->
-        <xacro:motor name = "${name}_right_shoulder" axis = "1 0 0" fixed_parent = "${hubName}" revolute_child = "${upperName}">
-            <origin xyz = "0 0 -0.005" rpy = "0 0 0"/>
-            <origin xyz = "0 0 -0.02" rpy = "0 ${PI/2} 0"/>
-        </xacro:motor>
         <!-- Create the covering for the upper portion of the leg -->
         <xacro:property name = "upperCoverName" value = "${name}_right_leg_cover"/>
@@ -90,4 +85,14 @@
             </collision>
         </link>
+        <!-- Connect leg to parent with a motor -->
+        <xacro:motor name = "${name}_right_shoulder_1" axis = "-1 0 0" fixed_parent = "${parent}" revolute_child = "${hubName}">
+            <xacro:insert_block name = "origin"/>
+            <origin xyz = "0 0 0.036" rpy = "0 ${PI/2} 0"/>
+        </xacro:motor>
+        <!-- Join the Hub and the Upper Link with a motor -->
+        <xacro:motor name = "${name}_right_shoulder_2" axis = "1 0 0" fixed_parent = "${hubName}" revolute_child = "${upperName}">
+            <origin xyz = "0 0 -0.005" rpy = "0 0 0"/>
+            <origin xyz = "0 0 -0.02" rpy = "0 ${PI/2} 0"/>
+        </xacro:motor>
         <!-- Connect Upper Link and Lower Link with a motor -->
         <xacro:motor name = "${name}_right_elbow" axis = "0 0 -1" fixed_parent = "${upperName}" revolute_child = "${lowerName}">
@@ -95,9 +100,4 @@
             <origin xyz = "0 0 -0.032" rpy = "${PI} 0 0"/>
         </xacro:motor>
-        <!-- Connect leg to parent with a motor -->
-        <xacro:motor name = "${name}_right_parent_motor" axis = "-1 0 0" fixed_parent = "${parent}" revolute_child = "${hubName}">
-            <xacro:insert_block name = "origin"/>
-            <origin xyz = "0 0 0.036" rpy = "0 ${PI/2} 0"/>
-        </xacro:motor>
     </xacro:macro>
 </robot>

Commit message: Added feet to the model

File: pupper_description/left_leg.xacro (robot description, xacro)
@@ -85,4 +85,27 @@
             </collision>
         </link>
+        <!-- Create the foot pad -->
+        <link name = "${name}_left_foot">
+            <inertial>
+                <xacro:footInertia/>
+            </inertial>
+            <visual name = "${name}_left_foot_visual">
+                <material name = "red"/>
+                <geometry>
+                    <mesh filename = "${VisualPath}/Leg/hemisphere.stl" scale = "0.00026 0.00026 0.00026"/>
+                </geometry>
+            </visual>
+            <collision name = "${name}_left_foot_collision">
+                <geometry>
+                    <mesh filename = "${CollisionPath}/Leg/hemisphere_simplified.dae" scale = "0.00026 0.00026 0.00026"/>
+                </geometry>
+            </collision>
+        </link>
+        <!-- Connect foot pad to lower link -->
+        <joint name = "${name}_left_foot_joint" type = "fixed">
+            <parent link = "${lowerName}"/>
+            <child  link = "${name}_left_foot"/>
+            <origin xyz = "0 -0.11 0.009" rpy = "${PI/2} 0 ${PI/4 - 0.1}"/>
+        </joint>
         <!-- Connect leg to parent with a motor -->
         <xacro:motor name = "${name}_left_shoulder_1" axis = "-1 0 0" fixed_parent = "${parent}" revolute_child = "${hubName}">

File: pupper_description/pupper.urdf.xacro (robot description, xacro)
@@ -12,5 +12,5 @@
     <xacro:property name = "meshScale_in"  value = "0.0254 0.0254 0.0254"/>
     <xacro:property name = "massScale"     value = "${1240/(1000**3)}"/>    <!-- Convert mm^3 to kg-->
-    <xacro:property name = "density"       value = "1240"/>                 <!-- NOTE: density in kg/m^3 -->
+    <xacro:property name = "density"       value = "${1240*0.3}"/>                 <!-- NOTE: density in kg/m^3 -->
     <xacro:property name = "inch2meter"    value = "${25.4/1000}"/>
     <xacro:property name = "inch2mm"       value = "25.4"/>
@@ -25,8 +25,16 @@
                  ixy = "${ixy*kConvert}" iyz = "${iyz*kConvert}" ixz = "${ixz*kConvert}"/>
     </xacro:macro>
+    <xacro:macro name = "footInertia">
+        <xacro:property name = "foot_mass" value = "0.01"/>
+        <xacro:property name = "foot_radius" value = "0.0095"/>
+        <xacro:property name = "i__" value = "${2/5 * foot_mass * foot_radius**2}"/>
+        <mass value = "${foot_mass}"/>
+        <inertia ixx = "${i__}" iyy = "${i__}" izz = "${i__}" ixy = "0" ixz = "0" iyz = "0"/>
+    </xacro:macro>
     <!-- Connect the plugin -->
     <gazebo>
         <plugin filename = "libpupper_plugin.so" name = "pupper_plugin"/>
     </gazebo>
+    <!-- TODO: Get the correct mass and inertia on the feet -->
     <!-- ++++++++++++++++ -->
     <!-- ROBOT START HERE -->

File: pupper_description/right_leg.xacro (robot description, xacro)
@@ -85,4 +85,27 @@
             </collision>
         </link>
+        <!-- Create the foot pad -->
+        <link name = "${name}_right_foot">
+            <inertial>
+                <xacro:footInertia/>
+            </inertial>
+            <visual name = "${name}_right_foot_visual">
+                <material name = "red"/>
+                <geometry>
+                    <mesh filename = "${VisualPath}/Leg/hemisphere.stl" scale = "0.00026 0.00026 0.00026"/>
+                </geometry>
+            </visual>
+            <collision name = "${name}_right_foot_collision">
+                <geometry>
+                    <mesh filename = "${CollisionPath}/Leg/hemisphere_simplified.dae" scale = "0.00026 0.00026 0.00026"/>
+                </geometry>
+            </collision>
+        </link>
+        <!-- Connect foot pad to lower link -->
+        <joint name = "${name}_right_foot_joint" type = "fixed">
+            <parent link = "${lowerName}"/>
+            <child  link = "${name}_right_foot"/>
+            <origin xyz = "0 -0.11 -0.009" rpy = "${PI/2} 0 ${PI/4 - 0.1}"/>
+        </joint>
         <!-- Connect leg to parent with a motor -->
         <xacro:motor name = "${name}_right_shoulder_1" axis = "-1 0 0" fixed_parent = "${parent}" revolute_child = "${hubName}">

Commit message: Fixed the https://www.youtube.com/watch?v=Kmp5dgzeZuk

File: pupper_description/left_leg.xacro (robot description, xacro)
@@ -102,4 +102,15 @@
             </collision>
         </link>
+        <gazebo reference = "${lowerName}">
+            <collision name = "${lowerName}_collision">
+                <surface>
+                    <contact>
+                        <ode>
+                            <min_depth>0.01</min_depth>
+                        </ode>
+                    </contact>
+                </surface>
+            </collision>
+        </gazebo>
         <!-- Connect foot pad to lower link -->
         <joint name = "${name}_left_foot_joint" type = "fixed">

File: pupper_description/motor.xacro (robot description, xacro)
@@ -36,5 +36,5 @@
             <xacro:insert_block name = "revolute_origin"/>
             <limit upper = "1e10" lower = "-1e10" effort = "1e6" velocity = "1e6"/>
-            <dynamics damping = "0.3" friction = "0.1"/>
+            <dynamics damping = "0.3" friction = "0.3"/>
             <axis xyz = "${axis}"/>
         </joint>
@@ -42,7 +42,15 @@
         <!-- provideFeedback     : allows the joint to publish torque data -->
         <gazebo reference = "${name}_joint">
+            <physics>
+                <ode>
+                    <max_force>50</max_force>
+                </ode>
+            </physics>
             <provideFeedback>true</provideFeedback>
             <implicitSpringDamper>true</implicitSpringDamper>
         </gazebo>
+        <gazebo reference = "${revolute_child}">
+            <self_collide>true</self_collide>
+        </gazebo>
     </xacro:macro>
 </robot>

File: pupper_description/pupper.urdf.xacro (robot description, xacro)
@@ -221,4 +221,5 @@
         </visual>
     </link>
+    <!-- Connect battery to body -->
     <joint name = "battery_to_body" type = "fixed">
         <parent link = "bottom_PCB"/>

File: pupper_description/right_leg.xacro (robot description, xacro)
@@ -102,4 +102,15 @@
             </collision>
         </link>
+        <gazebo reference = "${lowerName}">
+            <collision name = "${lowerName}_collision">
+                <surface>
+                    <contact>
+                        <ode>
+                            <min_depth>0.01</min_depth>
+                        </ode>
+                    </contact>
+                </surface>
+            </collision>
+        </gazebo>
         <!-- Connect foot pad to lower link -->
         <joint name = "${name}_right_foot_joint" type = "fixed">
@@ -119,5 +130,5 @@
         </xacro:motor>
         <!-- Connect Upper Link and Lower Link with a motor -->
-        <xacro:motor name = "${name}_right_elbow" axis = "0 0 -1" fixed_parent = "${upperName}" revolute_child = "${lowerName}">
+        <xacro:motor name = "${name}_right_elbow" axis = "0 0 1" fixed_parent = "${upperName}" revolute_child = "${lowerName}">
             <origin xyz = "0.023 0.082 0" rpy = "0 ${PI/2} 0"/>
             <origin xyz = "0 0 -0.032" rpy = "${PI} 0 0"/>
