Commit message: Renamed URDF joints and links to be more consistent

File: pupper_description/left_leg.xacro (robot description, xacro)
@@ -4,5 +4,5 @@
     <xacro:macro name = "leftLeg" params = "name parent *origin">
         <!-- Create hub that connects to the motor -->
-        <xacro:property name = "hubName" value = "${name}_left_leg_hub"/>
+        <xacro:property name = "hubName" value = "${name}_left_hub"/>
         <link name = "${hubName}">
             <inertial>
@@ -10,4 +10,5 @@
                 <xacro:scaleInertia ixx = "1456709" ixz = "446692" iyy = "1472451" izz = "1155732"/>
             </inertial>
+            <xacro:if value = "${full_urdf}">
             <visual name = "${hubName}_visual">
                 <material name = "blue"/>
@@ -21,7 +22,8 @@
                 </geometry>
             </collision>
+            </xacro:if>
         </link>
         <!-- Create the upper link portion (the thigh, if you will) -->
-        <xacro:property name = "upperName" value = "${name}_left_leg_upper_link"/>
+        <xacro:property name = "upperName" value = "${name}_left_upper_link"/>
         <link name = "${upperName}">
             <inertial>
@@ -29,4 +31,5 @@
                 <xacro:scaleInertia ixx = "14050550" ixy = "156735" iyy = "957647" izz = "13227597"/>
             </inertial>
+            <xacro:if value = "${full_urdf}">
             <visual name = "${upperName}_visual">
                 <material name = "yellow"/>
@@ -40,7 +43,8 @@
                 </geometry>
             </collision>
+            </xacro:if>
         </link>
         <!-- Create the covering for the upper portion of the leg -->
-        <xacro:property name = "upperCoverName" value = "${name}_left_leg_cover"/>
+        <xacro:property name = "upperCoverName" value = "${name}_left_cover"/>
         <link name = "${upperCoverName}">
             <inertial>
@@ -48,4 +52,5 @@
                 <xacro:scaleInertia ixx = "4268927" iyy = "991662" izz = "3827615" ixy = "171794" ixz = "0.7" iyz = "-24"/>
             </inertial>
+            <xacro:if value = "${full_urdf}">
             <visual name = "${upperCoverName}_visual">
                 <material name = "red"/>
@@ -59,4 +64,5 @@
                 </geometry>
             </collision>
+            </xacro:if>
         </link>
         <!-- Connect the covering to the upper link -->
@@ -67,5 +73,5 @@
         </joint>
         <!-- Creat the lower link -->
-        <xacro:property name = "lowerName" value = "${name}_lower_left_link"/>
+        <xacro:property name = "lowerName" value = "${name}_left_lower_link"/>
         <link name = "${lowerName}">
             <inertial>
@@ -73,4 +79,5 @@
                 <xacro:scaleInertia ixx = "18151954" iyy = "437604" izz = "18307054" ixy = "-238617" ixz = "19947" iyz = "672611"/>
             </inertial>
+            <xacro:if value = "${full_urdf}">
             <visual>
                 <material name = "blueGreen"/>
@@ -84,4 +91,5 @@
                 </geometry>
             </collision>
+            </xacro:if>
         </link>
         <!-- Create the foot pad -->
@@ -90,4 +98,5 @@
                 <xacro:footInertia/>
             </inertial>
+            <xacro:if value = "${full_urdf}">
             <visual name = "${name}_left_foot_visual">
                 <material name = "red"/>
@@ -101,5 +110,7 @@
                 </geometry>
             </collision>
+            </xacro:if>
         </link>
+        <xacro:if value = "${full_urdf}">
         <gazebo reference = "${lowerName}">
             <collision name = "${lowerName}_collision">
@@ -113,4 +124,5 @@
             </collision>
         </gazebo>
+        </xacro:if>
         <!-- Connect foot pad to lower link -->
         <joint name = "${name}_left_foot_joint" type = "fixed">
@@ -120,10 +132,10 @@
         </joint>
         <!-- Connect leg to parent with a motor -->
-        <xacro:motor name = "${name}_left_shoulder_1" axis = "-1 0 0" fixed_parent = "${parent}" revolute_child = "${hubName}">
+        <xacro:motor name = "${name}_left_hip" axis = "-1 0 0" fixed_parent = "${parent}" revolute_child = "${hubName}">
             <xacro:insert_block name = "origin"/>
             <origin xyz = "0 0 0.036" rpy = "0 ${PI/2} 0"/>
         </xacro:motor>
         <!-- Join the Hub and the Upper Link with a motor -->
-        <xacro:motor name = "${name}_left_shoulder_2" axis = "1 0 0" fixed_parent = "${hubName}" revolute_child = "${upperName}">
+        <xacro:motor name = "${name}_left_shoulder" axis = "1 0 0" fixed_parent = "${hubName}" revolute_child = "${upperName}">
             <origin xyz = "0 0 0.005" rpy = "0 0 0"/>
             <origin xyz = "0 0 0.022" rpy = "0 ${-PI/2} 0"/>

File: pupper_description/motor.xacro (robot description, xacro)
@@ -10,4 +10,5 @@
                 <inertia ixx = "7.2e-6" iyy = "1.11e-5" izz = "1.11e-5" ixy = "0" ixz = "0" iyz = "0"/>
             </inertial>
+            <xacro:if value = "${full_urdf}">
             <visual name = "${name}_visual">
                 <material name = "motorColor">
@@ -23,4 +24,5 @@
                 </geometry>
             </collision>
+            </xacro:if>
         </link>
         <!-- Rigidly attach to motor to it's parent -->
@@ -39,4 +41,5 @@
             <axis xyz = "${axis}"/>
         </joint>
+        <xacro:if value = "${full_urdf}">
         <!-- implicitSpringDamper: prevent crashing when damping is set -->
         <!-- provideFeedback     : allows the joint to publish torque data -->
@@ -53,4 +56,5 @@
             <self_collide>true</self_collide>
         </gazebo>
+        </xacro:if>
     </xacro:macro>
 </robot>

File: pupper_description/pupper.urdf (robot description, URDF)
Before this commit: robot pupper, 41 links, 40 joints
Links:
- removed link back_left_leg_cover
- removed link back_left_leg_hub
- removed link back_left_leg_upper_link
- removed link back_left_shoulder_1
- removed link back_left_shoulder_2
- removed link back_lower_left_link
- removed link back_lower_right_link
- removed link back_right_leg_cover
- removed link back_right_leg_hub
- removed link back_right_leg_upper_link
- removed link back_right_shoulder_1
- removed link back_right_shoulder_2
- removed link front_left_leg_cover
- removed link front_left_leg_hub
- removed link front_left_leg_upper_link
- removed link front_left_shoulder_1
- removed link front_left_shoulder_2
- removed link front_lower_left_link
- removed link front_lower_right_link
- removed link front_right_leg_cover
- removed link front_right_leg_hub
- removed link front_right_leg_upper_link
- removed link front_right_shoulder_1
- removed link front_right_shoulder_2
- added link back_left_cover, mass 0.002386008; collision mesh filename=package://ase389/pupper_description/Pupper_STL/Leg/part3_sh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 scale=0.001 0.001 0.001; visual mesh filename=package://ase389/pupper_description/Pupper_STL/Leg/part3_sh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 scale=0.001 0.001 0.001
- added link back_left_hip, mass 0.12; collision cylinder length=0.03 radius=0.012; visual cylinder length=0.03 radius=0.012
- added link back_left_hub, mass 0.002639712; collision mesh filename=package://ase389/pupper_description/Pupper_STL/Leg/part1_hu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 scale=0.001 0.001 0.001; visual mesh filename=package://ase389/pupper_description/Pupper_STL/Leg/part1_hu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 scale=0.001 0.001 0.001
- added link back_left_lower_link, mass 0.00489924; collision mesh filename=package://ase389/pupper_description/Pupper_STL/Leg/part4_lo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 scale=0.001 0.001 0.001; visual mesh filename=package://ase389/pupper_description/Pupper_STL/Leg/part4_lo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 scale=0.001 0.001 0.001
- added link back_left_shoulder, mass 0.12; collision cylinder length=0.03 radius=0.012; visual cylinder length=0.03 radius=0.012
- added link back_left_upper_link, mass 0.005135088; collision mesh filename=package://ase389/pupper_description/Pupper_STL/Leg/part2_up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 scale=0.001 0.001 0.001; visual mesh filename=package://ase389/pupper_description/Pupper_STL/Leg/part2_up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 scale=0.001 0.001 0.001
- added link back_right_cover, mass 0.002386008; collision mesh filename=package://ase389/pupper_description/Pupper_STL/Leg/part3_sh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 scale=0.001 0.001 0.001; visual mesh filename=package://ase389/pupper_description/Pupper_STL/Leg/part3_sh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 scale=0.001 0.001 0.001
- added link back_right_hip, mass 0.12; collision cylinder length=0.03 radius=0.012; visual cylinder length=0.03 radius=0.012
- added link back_right_hub, mass 0.002639712; collision mesh filename=package://ase389/pupper_description/Pupper_STL/Leg/part1_hu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 scale=0.001 0.001 0.001; visual mesh filename=package://ase389/pupper_description/Pupper_STL/Leg/part1_hu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 scale=0.001 0.001 0.001
- added link back_right_lower_link, mass 0.00489924; collision mesh filename=package://ase389/pupper_description/Pupper_STL/Leg/part4_lo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 scale=0.001 0.001 0.001; visual mesh filename=package://ase389/pupper_description/Pupper_STL/Leg/part4_lo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 scale=0.001 0.001 0.001
- added link back_right_shoulder, mass 0.12; collision cylinder length=0.03 radius=0.012; visual cylinder length=0.03 radius=0.012
- added link back_right_upper_link, mass 0.005135088; collision mesh filename=package://ase389/pupper_description/Pupper_STL/Leg/part2_up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 scale=0.001 0.001 0.001; visual mesh filename=package://ase389/pupper_description/Pupper_STL/Leg/part2_up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 scale=0.001 0.001 0.001
- added link front_left_cover, mass 0.002386008; collision mesh filename=package://ase389/pupper_description/Pupper_STL/Leg/part3_sh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 scale=0.001 0.001 0.001; visual mesh filename=package://ase389/pupper_description/Pupper_STL/Leg/part3_sh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 scale=0.001 0.001 0.001
- added link front_left_hip, mass 0.12; collision cylinder length=0.03 radius=0.012; visual cylinder length=0.03 radius=0.012
- added link front_left_hub, mass 0.002639712; collision mesh filename=package://ase389/pupper_description/Pupper_STL/Leg/part1_hu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 scale=0.001 0.001 0.001; visual mesh filename=package://ase389/pupper_description/Pupper_STL/Leg/part1_hu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 scale=0.001 0.001 0.001
- added link front_left_lower_link, mass 0.00489924; collision mesh filename=package://ase389/pupper_description/Pupper_STL/Leg/part4_lo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 scale=0.001 0.001 0.001; visual mesh filename=package://ase389/pupper_description/Pupper_STL/Leg/part4_lo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 scale=0.001 0.001 0.001
- added link front_left_shoulder, mass 0.12; collision cylinder length=0.03 radius=0.012; visual cylinder length=0.03 radius=0.012
- added link front_left_upper_link, mass 0.005135088; collision mesh filename=package://ase389/pupper_description/Pupper_STL/Leg/part2_up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 scale=0.001 0.001 0.001; visual mesh filename=package://ase389/pupper_description/Pupper_STL/Leg/part2_up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 scale=0.001 0.001 0.001
- added link front_right_cover, mass 0.002386008; collision mesh filename=package://ase389/pupper_description/Pupper_STL/Leg/part3_sh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 scale=0.001 0.001 0.001; visual mesh filename=package://ase389/pupper_description/Pupper_STL/Leg/part3_sh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 scale=0.001 0.001 0.001
- added link front_right_hip, mass 0.12; collision cylinder length=0.03 radius=0.012; visual cylinder length=0.03 radius=0.012
- added link front_right_hub, mass 0.002639712; collision mesh filename=package://ase389/pupper_description/Pupper_STL/Leg/part1_hu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 scale=0.001 0.001 0.001; visual mesh filename=package://ase389/pupper_description/Pupper_STL/Leg/part1_hu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 scale=0.001 0.001 0.001
- added link front_right_lower_link, mass 0.00489924; collision mesh filename=package://ase389/pupper_description/Pupper_STL/Leg/part4_lo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 scale=0.001 0.001 0.001; visual mesh filename=package://ase389/pupper_description/Pupper_STL/Leg/part4_lo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 scale=0.001 0.001 0.001
- added link front_right_shoulder, mass 0.12; collision cylinder length=0.03 radius=0.012; visual cylinder length=0.03 radius=0.012
- added link front_right_upper_link, mass 0.005135088; collision mesh filename=package://ase389/pupper_description/Pupper_STL/Leg/part2_up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 scale=0.001 0.001 0.001; visual mesh filename=package://ase389/pupper_description/Pupper_STL/Leg/part2_up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 scale=0.001 0.001 0.001
Joints:
- removed joint back_left_shoulder_1_fixed_joint
- removed joint back_left_shoulder_1_joint
- removed joint back_left_shoulder_2_fixed_joint
- removed joint back_left_shoulder_2_joint
- removed joint back_right_shoulder_1_fixed_joint
- removed joint back_right_shoulder_1_joint
- removed joint back_right_shoulder_2_fixed_joint
- removed joint back_right_shoulder_2_joint
- removed joint front_left_shoulder_1_fixed_joint
- removed joint front_left_shoulder_1_joint
- removed joint front_left_shoulder_2_fixed_joint
- removed joint front_left_shoulder_2_joint
- removed joint front_right_shoulder_1_fixed_joint
- removed joint front_right_shoulder_1_joint
- removed joint front_right_shoulder_2_fixed_joint
- removed joint front_right_shoulder_2_joint
- added joint back_left_hip_fixed_joint: type fixed, parent bottom_PCB, child back_left_hip, origin xyz=0.05 0.095 0.044 rpy=-1.5707963268 0 0
- added joint back_left_hip_joint: type revolute, parent back_left_hip, child back_left_hub, origin xyz=0 0 0.036 rpy=0 1.5707963268 0, axis -1 0 0, limit lower=-1e10 upper=1e10 effort=1e6 velocity=1e6
- added joint back_left_shoulder_fixed_joint: type fixed, parent back_left_hub, child back_left_shoulder, origin xyz=0 0 0.005 rpy=0 0 0
- added joint back_left_shoulder_joint: type revolute, parent back_left_shoulder, child back_left_upper_link, origin xyz=0 0 0.022 rpy=0 -1.5707963268 0, axis 1 0 0, limit lower=-1e10 upper=1e10 effort=1e6 velocity=1e6
- added joint back_right_hip_fixed_joint: type fixed, parent bottom_PCB, child back_right_hip, origin xyz=-0.045 0.095 0.044 rpy=-1.5707963268 0 0
- added joint back_right_hip_joint: type revolute, parent back_right_hip, child back_right_hub, origin xyz=0 0 0.036 rpy=0 1.5707963268 0, axis -1 0 0, limit lower=-1e10 upper=1e10 effort=1e6 velocity=1e6
- added joint back_right_shoulder_fixed_joint: type fixed, parent back_right_hub, child back_right_shoulder, origin xyz=0 0 -0.005 rpy=0 0 0
- added joint back_right_shoulder_joint: type revolute, parent back_right_shoulder, child back_right_upper_link, origin xyz=0 0 -0.02 rpy=0 1.5707963268 0, axis 1 0 0, limit lower=-1e10 upper=1e10 effort=1e6 velocity=1e6
- added joint front_left_hip_fixed_joint: type fixed, parent bottom_PCB, child front_left_hip, origin xyz=0.05 -0.105 0.044 rpy=-1.5707963268 0 0
- added joint front_left_hip_joint: type revolute, parent front_left_hip, child front_left_hub, origin xyz=0 0 0.036 rpy=0 1.5707963268 0, axis -1 0 0, limit lower=-1e10 upper=1e10 effort=1e6 velocity=1e6
- added joint front_left_shoulder_fixed_joint: type fixed, parent front_left_hub, child front_left_shoulder, origin xyz=0 0 0.005 rpy=0 0 0
- added joint front_left_shoulder_joint: type revolute, parent front_left_shoulder, child front_left_upper_link, origin xyz=0 0 0.022 rpy=0 -1.5707963268 0, axis 1 0 0, limit lower=-1e10 upper=1e10 effort=1e6 velocity=1e6
- added joint front_right_hip_fixed_joint: type fixed, parent bottom_PCB, child front_right_hip, origin xyz=-0.045 -0.105 0.044 rpy=-1.5707963268 0 0
- added joint front_right_hip_joint: type revolute, parent front_right_hip, child front_right_hub, origin xyz=0 0 0.036 rpy=0 1.5707963268 0, axis -1 0 0, limit lower=-1e10 upper=1e10 effort=1e6 velocity=1e6
- added joint front_right_shoulder_fixed_joint: type fixed, parent front_right_hub, child front_right_shoulder, origin xyz=0 0 -0.005 rpy=0 0 0
- added joint front_right_shoulder_joint: type revolute, parent front_right_shoulder, child front_right_upper_link, origin xyz=0 0 -0.02 rpy=0 1.5707963268 0, axis 1 0 0, limit lower=-1e10 upper=1e10 effort=1e6 velocity=1e6
- joint back_left_elbow_fixed_joint: parent back_left_leg_upper_link -> back_left_upper_link
- joint back_left_elbow_joint: child back_lower_left_link -> back_left_lower_link
- joint back_left_foot_joint: parent back_lower_left_link -> back_left_lower_link
- joint back_left_shroud_to_leg: child back_left_leg_cover -> back_left_cover; parent back_left_leg_upper_link -> back_left_upper_link
- joint back_right_elbow_fixed_joint: parent back_right_leg_upper_link -> back_right_upper_link
- joint back_right_elbow_joint: child back_lower_right_link -> back_right_lower_link
- joint back_right_foot_joint: parent back_lower_right_link -> back_right_lower_link
- joint back_right_shroud_to_leg: child back_right_leg_cover -> back_right_cover; parent back_right_leg_upper_link -> back_right_upper_link
- joint front_left_elbow_fixed_joint: parent front_left_leg_upper_link -> front_left_upper_link
- joint front_left_elbow_joint: child front_lower_left_link -> front_left_lower_link
- joint front_left_foot_joint: parent front_lower_left_link -> front_left_lower_link
- joint front_left_shroud_to_leg: child front_left_leg_cover -> front_left_cover; parent front_left_leg_upper_link -> front_left_upper_link
- joint front_right_elbow_fixed_joint: parent front_right_leg_upper_link -> front_right_upper_link
- joint front_right_elbow_joint: child front_lower_right_link -> front_right_lower_link
- joint front_right_foot_joint: parent front_lower_right_link -> front_right_lower_link
- joint front_right_shroud_to_leg: child front_right_leg_cover -> front_right_cover; parent front_right_leg_upper_link -> front_right_upper_link

File: pupper_description/pupper.urdf.xacro (robot description, xacro)
@@ -1,6 +1,9 @@
 <?xml version="1.0"?>
 <robot name = "pupper" xmlns:xacro="http://www.ros.org/wiki/xacro">
+    <xacro:property name = "full_urdf" value = "true"/>
+    <xacro:if value = "${full_urdf}">
+    <xacro:include filename = "$(find ase389)/pupper_description/colors.xacro"/>
+    </xacro:if>
     <xacro:include filename = "$(find ase389)/pupper_description/motor.xacro"/>
-    <xacro:include filename = "$(find ase389)/pupper_description/colors.xacro"/>
     <xacro:include filename = "$(find ase389)/pupper_description/left_leg.xacro"/>
     <xacro:include filename = "$(find ase389)/pupper_description/right_leg.xacro"/>
@@ -46,4 +49,5 @@
             <xacro:scaleInertia ixx = "41.05" iyy = "4.405" izz = "45.448" scaling_factor = "${inch2meter}"/>
         </inertial>
+        <xacro:if value = "${full_urdf}">
         <visual name = "bottom_PCB_visual">
             <geometry>
@@ -56,4 +60,5 @@
             </geometry>
         </collision>
+        </xacro:if>
     </link>
     <!-- Create Front bulkhead -->
@@ -63,4 +68,5 @@
             <xacro:scaleInertia ixx = "27491730" iyy = "74592784" izz = "83928296"/>
         </inertial>
+        <xacro:if value = "${full_urdf}">
         <visual>
             <material name = "red"/>
@@ -74,4 +80,5 @@
             </geometry>
         </collision>
+        </xacro:if>
     </link>
     <!-- Join Front Bulkhead with Base -->
@@ -87,4 +94,5 @@
             <xacro:scaleInertia ixx = "22996456" iyy = "51008240" izz = "73639128"/>
         </inertial>
+        <xacro:if value = "${full_urdf}">
         <visual name = "middle_bulkhead_front_visual">
             <material name = "blue"/>
@@ -98,4 +106,5 @@
             </geometry>
         </collision>
+        </xacro:if>
     </link>
     <!-- Join Middle Bulkhead to Base -->
@@ -111,4 +120,5 @@
             <xacro:scaleInertia ixx = "21912060" iyy = "40583024" izz = "62043808"/>
         </inertial>
+        <xacro:if value = "${full_urdf}">
         <visual name = "middle_bulkhead_rear_visual">
             <material name = "blue"/>
@@ -122,4 +132,5 @@
             </geometry>
         </collision>
+        </xacro:if>
     </link>
     <!-- Join 2nd Bulkhead to Base -->
@@ -135,4 +146,5 @@
             <xacro:scaleInertia ixx = "30641556" iyy = "21280556" izz = "10692993"/>
         </inertial>
+        <xacro:if value = "${full_urdf}">
         <visual name = "back_right_shroud_visual">
             <material name = "yellow"/>
@@ -146,4 +158,5 @@
             </geometry>
         </collision>
+        </xacro:if>
     </link>
     <!-- Connect back right shroud to body -->
@@ -159,4 +172,5 @@
             <xacro:scaleInertia ixx = "30641502" iyy = "21280568" izz = "10692940"/>
         </inertial>
+        <xacro:if value = "${full_urdf}">
         <visual name = "back_left_shroud_visual">
             <material name = "yellow"/>
@@ -171,4 +185,5 @@
             </geometry>
         </collision>
+        </xacro:if>
     </link>
     <!-- Join back left shroud to body -->
@@ -184,4 +199,5 @@
             <xacro:scaleInertia ixx = "23357426" iyy = "52151916" iyz = "-17892" izz = "75135296"/>
         </inertial>
+        <xacro:if value = "${full_urdf}">
         <visual>
             <material name = "blue"/>
@@ -195,4 +211,5 @@
             </geometry>
         </collision>
+        </xacro:if>
     </link>
     <!-- Join rear bulkhead to body -->
@@ -214,4 +231,5 @@
                      izz = "${1/12 * batt_m * (batt_x**2 + batt_y**2)}"/>
         </inertial>
+        <xacro:if value = "${full_urdf}">
         <visual name = "battery_visual">
             <material name = "pink"/>
@@ -220,4 +238,5 @@
             </geometry>
         </visual>
+        </xacro:if>
     </link>
     <!-- Connect battery to body -->
@@ -233,4 +252,5 @@
             <xacro:scaleInertia ixx = "41.05" iyy = "4.405" izz = "45.448" scaling_factor = "${inch2meter}"/>
         </inertial>
+        <xacro:if value = "${full_urdf}">
         <visual name = "top_PCB_visual">
             <geometry>
@@ -243,4 +263,5 @@
             </geometry>
         </collision>
+        </xacro:if>
     </link>
     <!-- Joint top plate to body -->
