Commit message: Renamed URDF joints and links to be more consistent

File: pupper_description/right_leg.xacro (robot description, xacro)
@@ -4,5 +4,5 @@
     <xacro:macro name = "rightLeg" params = "name parent *origin">
         <!-- Create hub that connects to the motor -->
-        <xacro:property name = "hubName" value = "${name}_right_leg_hub"/>
+        <xacro:property name = "hubName" value = "${name}_right_hub"/>
         <link name = "${hubName}">
             <inertial>
@@ -10,4 +10,5 @@
                 <xacro:scaleInertia ixx = "1456709" ixz = "-446692" iyy = "1472451" izz = "1155732"/>
             </inertial>
+            <xacro:if value = "${full_urdf}">
             <visual name = "${hubName}_visual">
                 <material name = "blue"/>
@@ -21,7 +22,8 @@
                 </geometry>
             </collision>
+            </xacro:if>
         </link>
         <!-- Create the upper link portion (the thigh, if you will) -->
-        <xacro:property name = "upperName" value = "${name}_right_leg_upper_link"/>
+        <xacro:property name = "upperName" value = "${name}_right_upper_link"/>
         <link name = "${upperName}">
             <inertial>
@@ -29,4 +31,5 @@
                 <xacro:scaleInertia ixx = "14050550" ixy = "156735" iyy = "957647" izz = "13227597"/>
             </inertial>
+            <xacro:if value = "${full_urdf}">
             <visual name = "${upperName}_visual">
                 <material name = "yellow"/>
@@ -40,7 +43,8 @@
                 </geometry>
             </collision>
+            </xacro:if>
         </link>
         <!-- Create the covering for the upper portion of the leg -->
-        <xacro:property name = "upperCoverName" value = "${name}_right_leg_cover"/>
+        <xacro:property name = "upperCoverName" value = "${name}_right_cover"/>
         <link name = "${upperCoverName}">
             <inertial>
@@ -48,4 +52,5 @@
                 <xacro:scaleInertia ixx = "4268927" iyy = "991662" izz = "3827615" ixy = "171794" ixz = "0.7" iyz = "-24"/>
             </inertial>
+            <xacro:if value = "${full_urdf}">
             <visual name = "${upperCoverName}_visual">
                 <material name = "red"/>
@@ -59,4 +64,5 @@
                 </geometry>
             </collision>
+            </xacro:if>
         </link>
         <!-- Connect the covering to the upper link -->
@@ -67,5 +73,5 @@
         </joint>
         <!-- Creat the lower link -->
-        <xacro:property name = "lowerName" value = "${name}_lower_right_link"/>
+        <xacro:property name = "lowerName" value = "${name}_right_lower_link"/>
         <link name = "${lowerName}">
             <inertial>
@@ -73,4 +79,5 @@
                 <xacro:scaleInertia ixx = "18151954" iyy = "437604" izz = "18307054" ixy = "-238617" ixz = "-19947" iyz = "-672611"/>
             </inertial>
+            <xacro:if value = "${full_urdf}">
             <visual>
                 <material name = "blueGreen"/>
@@ -84,4 +91,5 @@
                 </geometry>
             </collision>
+            </xacro:if>
         </link>
         <!-- Create the foot pad -->
@@ -90,4 +98,5 @@
                 <xacro:footInertia/>
             </inertial>
+            <xacro:if value = "${full_urdf}">
             <visual name = "${name}_right_foot_visual">
                 <material name = "red"/>
@@ -101,5 +110,7 @@
                 </geometry>
             </collision>
+            </xacro:if>
         </link>
+        <xacro:if value = "${full_urdf}">
         <gazebo reference = "${lowerName}">
             <collision name = "${lowerName}_collision">
@@ -113,4 +124,5 @@
             </collision>
         </gazebo>
+        </xacro:if>
         <!-- Connect foot pad to lower link -->
         <joint name = "${name}_right_foot_joint" type = "fixed">
@@ -120,10 +132,10 @@
         </joint>
         <!-- Connect leg to parent with a motor -->
-        <xacro:motor name = "${name}_right_shoulder_1" axis = "-1 0 0" fixed_parent = "${parent}" revolute_child = "${hubName}">
+        <xacro:motor name = "${name}_right_hip" axis = "-1 0 0" fixed_parent = "${parent}" revolute_child = "${hubName}">
             <xacro:insert_block name = "origin"/>
             <origin xyz = "0 0 0.036" rpy = "0 ${PI/2} 0"/>
         </xacro:motor>
         <!-- Join the Hub and the Upper Link with a motor -->
-        <xacro:motor name = "${name}_right_shoulder_2" axis = "1 0 0" fixed_parent = "${hubName}" revolute_child = "${upperName}">
+        <xacro:motor name = "${name}_right_shoulder" axis = "1 0 0" fixed_parent = "${hubName}" revolute_child = "${upperName}">
             <origin xyz = "0 0 -0.005" rpy = "0 0 0"/>
             <origin xyz = "0 0 -0.02" rpy = "0 ${PI/2} 0"/>

Commit message: Added contact detection in gazebo

File: pupper_description/left_leg.xacro (robot description, xacro)
@@ -112,17 +112,4 @@
             </xacro:if>
         </link>
-        <xacro:if value = "${full_urdf}">
-        <gazebo reference = "${lowerName}">
-            <collision name = "${lowerName}_collision">
-                <surface>
-                    <contact>
-                        <ode>
-                            <min_depth>0.01</min_depth>
-                        </ode>
-                    </contact>
-                </surface>
-            </collision>
-        </gazebo>
-        </xacro:if>
         <!-- Connect foot pad to lower link -->
         <joint name = "${name}_left_foot_joint" type = "fixed">

File: pupper_description/right_leg.xacro (robot description, xacro)
@@ -112,17 +112,4 @@
             </xacro:if>
         </link>
-        <xacro:if value = "${full_urdf}">
-        <gazebo reference = "${lowerName}">
-            <collision name = "${lowerName}_collision">
-                <surface>
-                    <contact>
-                        <ode>
-                            <min_depth>0.01</min_depth>
-                        </ode>
-                    </contact>
-                </surface>
-            </collision>
-        </gazebo>
-        </xacro:if>
         <!-- Connect foot pad to lower link -->
         <joint name = "${name}_right_foot_joint" type = "fixed">
