Commit message: Shifted joint parents to try to work with RBDL. Didn't work

File: pupper_description/left_leg.xacro (robot description, xacro)
@@ -2,5 +2,5 @@
 <robot name = "left_leg_macro" xmlns:xacro="http://www.ros.org/wiki/xacro">
     <!-- Macro for the creation of a leg -->
-    <xacro:macro name = "leftLeg" params = "name parent *origin">
+    <xacro:macro name = "leftLeg" params = "name parent *origin *origin2">
         <!-- Create hub that connects to the motor -->
         <xacro:property name = "hubName" value = "${name}_left_hub"/>
@@ -118,12 +118,16 @@
             <origin xyz = "0 -0.11 0.009" rpy = "${PI/2} 0 ${PI/4 - 0.1}"/>
         </joint>
+        <xacro:property name = "new_origin" value = "${origin}"/>
         <!-- Connect leg to parent with a motor -->
         <xacro:motor name = "${name}_left_hip" axis = "-1 0 0" fixed_parent = "${parent}" revolute_child = "${hubName}">
             <xacro:insert_block name = "origin"/>
-            <origin xyz = "0 0 0.036" rpy = "0 ${PI/2} 0"/>
+            <!-- <origin xyz = "0 0 0.036" rpy = "0 ${-PI/2} 0"/> -->
+            <!-- <origin xyz = "0 0.0 0.036" rpy = "${-PI/2} 0 0"/> -->
+            <xacro:insert_block name = "origin2"/>
         </xacro:motor>
         <!-- Join the Hub and the Upper Link with a motor -->
         <xacro:motor name = "${name}_left_shoulder" axis = "1 0 0" fixed_parent = "${hubName}" revolute_child = "${upperName}">
             <origin xyz = "0 0 0.005" rpy = "0 0 0"/>
+            <!-- <origin xyz = "0 0 0.022" rpy = "0 ${-PI/2} 0"/> -->
             <origin xyz = "0 0 0.022" rpy = "0 ${-PI/2} 0"/>
         </xacro:motor>
@@ -131,5 +135,6 @@
         <xacro:motor name = "${name}_left_elbow" axis = "0 0 -1" fixed_parent = "${upperName}" revolute_child = "${lowerName}">
             <origin xyz = "0.023 0.082 0" rpy = "0 ${PI/2} 0"/>
-            <origin xyz = "0 0 -0.032" rpy = "${PI} ${PI} 0"/>
+            <!-- <origin xyz = "0 0 -0.032" rpy = "${PI} ${PI} 0"/>  -->
+            <origin xyz = "-0.006 0.08 0" rpy = "0 ${-PI/2} ${PI}"/>
         </xacro:motor>
     </xacro:macro>

File: pupper_description/motor.xacro (robot description, xacro)
@@ -4,6 +4,7 @@
         <xacro:property name = "motorRad"    value = "0.012"/>
         <xacro:property name = "motorLength" value = "0.03"/>
+        <xacro:property name = "motorMass"   value = "0.120"/> <!-- kg -->
         <!-- Create the motor -->
-        <link name = "${name}">
+        <link name = "${name}_motor">
             <inertial>
                 <mass value = "0.12"/>
@@ -29,10 +30,11 @@
         <joint name = "${name}_fixed_joint" type = "fixed">
             <parent link = "${fixed_parent}"/>
-            <child  link = "${name}"/>
+            <child  link = "${name}_motor"/>
             <xacro:insert_block name = "fixed_origin"/>
         </joint>
         <!-- Attach the child link through a revolute joint -->
         <joint name = "${name}_joint" type = "revolute">
-            <parent link = "${name}"/>
+            <parent link = "${fixed_parent}"/>
+            <!-- <parent link = "${name}_motor"/> -->
             <child  link = "${revolute_child}"/>
             <xacro:insert_block name = "revolute_origin"/>

File: pupper_description/pupper.urdf (robot description, URDF)
Before this commit: robot pupper, 41 links, 40 joints
Links:
- removed link back_left_elbow
- removed link back_left_hip
- removed link back_left_shoulder
- removed link back_right_elbow
- removed link back_right_hip
- removed link back_right_shoulder
- removed link front_left_elbow
- removed link front_left_hip
- removed link front_left_shoulder
- removed link front_right_elbow
- removed link front_right_hip
- removed link front_right_shoulder
- added link back_left_elbow_motor, mass 0.12; collision cylinder length=0.03 radius=0.012; visual cylinder length=0.03 radius=0.012
- added link back_left_hip_motor, mass 0.12; collision cylinder length=0.03 radius=0.012; visual cylinder length=0.03 radius=0.012
- added link back_left_shoulder_motor, mass 0.12; collision cylinder length=0.03 radius=0.012; visual cylinder length=0.03 radius=0.012
- added link back_right_elbow_motor, mass 0.12; collision cylinder length=0.03 radius=0.012; visual cylinder length=0.03 radius=0.012
- added link back_right_hip_motor, mass 0.12; collision cylinder length=0.03 radius=0.012; visual cylinder length=0.03 radius=0.012
- added link back_right_shoulder_motor, mass 0.12; collision cylinder length=0.03 radius=0.012; visual cylinder length=0.03 radius=0.012
- added link front_left_elbow_motor, mass 0.12; collision cylinder length=0.03 radius=0.012; visual cylinder length=0.03 radius=0.012
- added link front_left_hip_motor, mass 0.12; collision cylinder length=0.03 radius=0.012; visual cylinder length=0.03 radius=0.012
- added link front_left_shoulder_motor, mass 0.12; collision cylinder length=0.03 radius=0.012; visual cylinder length=0.03 radius=0.012
- added link front_right_elbow_motor, mass 0.12; collision cylinder length=0.03 radius=0.012; visual cylinder length=0.03 radius=0.012
- added link front_right_hip_motor, mass 0.12; collision cylinder length=0.03 radius=0.012; visual cylinder length=0.03 radius=0.012
- added link front_right_shoulder_motor, mass 0.12; collision cylinder length=0.03 radius=0.012; visual cylinder length=0.03 radius=0.012
- link back_left_cover: geometry collision mesh filename=package://ase389/pupper_description/Pupper_STL/Leg/part3_sh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 scale=0.001 0.001 0.001; visual mesh filename=package://ase389/pupper_description/Pupper_STL/Leg/part3_sh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 scale=0.001 0.001 0.001
- link back_left_foot: geometry collision mesh filename=package://ase389/pupper_description/Pupper_STL/Leg/hemisphe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 scale=0.00026 0.00026 0.00026; visual mesh filename=package://ase389/pupper_description/Pupper_STL/Leg/hemisphe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 scale=0.00026 0.00026 0.00026
- link back_left_hub: geometry collision mesh filename=package://ase389/pupper_description/Pupper_STL/Leg/part1_hu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 scale=0.001 0.001 0.001; visual mesh filename=package://ase389/pupper_description/Pupper_STL/Leg/part1_hu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 scale=0.001 0.001 0.001
- link back_left_lower_link: geometry collision mesh filename=package://ase389/pupper_description/Pupper_STL/Leg/part4_lo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 scale=0.001 0.001 0.001; visual mesh filename=package://ase389/pupper_description/Pupper_STL/Leg/part4_lo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 scale=0.001 0.001 0.001
- link back_left_shroud: geometry collision mesh filename=package://ase389/pupper_description/Pupper_STL/Body/part5_l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 scale=0.001 0.001 0.001; visual mesh filename=package://ase389/pupper_description/Pupper_STL/Body/part5_l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 scale=0.001 0.001 0.001
- link back_left_upper_link: geometry collision mesh filename=package://ase389/pupper_description/Pupper_STL/Leg/part2_up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 scale=0.001 0.001 0.001; visual mesh filename=package://ase389/pupper_description/Pupper_STL/Leg/part2_up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 scale=0.001 0.001 0.001
- link back_right_cover: geometry collision mesh filename=package://ase389/pupper_description/Pupper_STL/Leg/part3_sh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 scale=0.001 0.001 0.001; visual mesh filename=package://ase389/pupper_description/Pupper_STL/Leg/part3_sh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 scale=0.001 0.001 0.001
- link back_right_foot: geometry collision mesh filename=package://ase389/pupper_description/Pupper_STL/Leg/hemisphe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 scale=0.00026 0.00026 0.00026; visual mesh filename=package://ase389/pupper_description/Pupper_STL/Leg/hemisphe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 scale=0.00026 0.00026 0.00026
- link back_right_hub: geometry collision mesh filename=package://ase389/pupper_description/Pupper_STL/Leg/part1_hu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 scale=0.001 0.001 0.001; visual mesh filename=package://ase389/pupper_description/Pupper_STL/Leg/part1_hu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 scale=0.001 0.001 0.001
- link back_right_lower_link: geometry collision mesh filename=package://ase389/pupper_description/Pupper_STL/Leg/part4_lo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 scale=0.001 0.001 0.001; visual mesh filename=package://ase389/pupper_description/Pupper_STL/Leg/part4_lo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 scale=0.001 0.001 0.001
- link back_right_shroud: geometry collision mesh filename=package://ase389/pupper_description/Pupper_STL/Body/part4_r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 scale=0.001 0.001 0.001; visual mesh filename=package://ase389/pupper_description/Pupper_STL/Body/part4_r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 scale=0.001 0.001 0.001
- link back_right_upper_link: geometry collision mesh filename=package://ase389/pupper_description/Pupper_STL/Leg/part2_up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 scale=0.001 0.001 0.001; visual mesh filename=package://ase389/pupper_description/Pupper_STL/Leg/part2_up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 scale=0.001 0.001 0.001
- link battery: geometry visual box size=0.07 0.035 0.0485
- link bottom_PCB: geometry collision mesh filename=package://ase389/pupper_description/Pupper_STL/Body/PCB_Boa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 scale=0.0254 0.0254 0.0254; visual mesh filename=package://ase389/pupper_description/Pupper_STL/Body/PCB_Boa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 scale=0.0254 0.0254 0.0254
- link front_bulkhead: geometry collision mesh filename=package://ase389/pupper_description/Pupper_STL/Body/part1_f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 scale=0.001 0.001 0.001; visual mesh filename=package://ase389/pupper_description/Pupper_STL/Body/part1_f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 scale=0.001 0.001 0.001
- link front_left_cover: geometry collision mesh filename=package://ase389/pupper_description/Pupper_STL/Leg/part3_sh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 scale=0.001 0.001 0.001; visual mesh filename=package://ase389/pupper_description/Pupper_STL/Leg/part3_sh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 scale=0.001 0.001 0.001
- link front_left_foot: geometry collision mesh filename=package://ase389/pupper_description/Pupper_STL/Leg/hemisphe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 scale=0.00026 0.00026 0.00026; visual mesh filename=package://ase389/pupper_description/Pupper_STL/Leg/hemisphe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 scale=0.00026 0.00026 0.00026
- link front_left_hub: geometry collision mesh filename=package://ase389/pupper_description/Pupper_STL/Leg/part1_hu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 scale=0.001 0.001 0.001; visual mesh filename=package://ase389/pupper_description/Pupper_STL/Leg/part1_hu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 scale=0.001 0.001 0.001
- link front_left_lower_link: geometry collision mesh filename=package://ase389/pupper_description/Pupper_STL/Leg/part4_lo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 scale=0.001 0.001 0.001; visual mesh filename=package://ase389/pupper_description/Pupper_STL/Leg/part4_lo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 scale=0.001 0.001 0.001
- link front_left_upper_link: geometry collision mesh filename=package://ase389/pupper_description/Pupper_STL/Leg/part2_up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 scale=0.001 0.001 0.001; visual mesh filename=package://ase389/pupper_description/Pupper_STL/Leg/part2_up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 scale=0.001 0.001 0.001
- link front_right_cover: geometry collision mesh filename=package://ase389/pupper_description/Pupper_STL/Leg/part3_sh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 scale=0.001 0.001 0.001; visual mesh filename=package://ase389/pupper_description/Pupper_STL/Leg/part3_sh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 scale=0.001 0.001 0.001
- link front_right_foot: geometry collision mesh filename=package://ase389/pupper_description/Pupper_STL/Leg/hemisphe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 scale=0.00026 0.00026 0.00026; visual mesh filename=package://ase389/pupper_description/Pupper_STL/Leg/hemisphe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 scale=0.00026 0.00026 0.00026
- link front_right_hub: geometry collision mesh filename=package://ase389/pupper_description/Pupper_STL/Leg/part1_hu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 scale=0.001 0.001 0.001; visual mesh filename=package://ase389/pupper_description/Pupper_STL/Leg/part1_hu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 scale=0.001 0.001 0.001
- link front_right_lower_link: geometry collision mesh filename=package://ase389/pupper_description/Pupper_STL/Leg/part4_lo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 scale=0.001 0.001 0.001; visual mesh filename=package://ase389/pupper_description/Pupper_STL/Leg/part4_lo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 scale=0.001 0.001 0.001
- link front_right_upper_link: geometry collision mesh filename=package://ase389/pupper_description/Pupper_STL/Leg/part2_up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 scale=0.001 0.001 0.001; visual mesh filename=package://ase389/pupper_description/Pupper_STL/Leg/part2_up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 scale=0.001 0.001 0.001
- link middle_bulkhead_front: geometry collision mesh filename=package://ase389/pupper_description/Pupper_STL/Body/part2_m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 scale=0.001 0.001 0.001; visual mesh filename=package://ase389/pupper_description/Pupper_STL/Body/part2_m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 scale=0.001 0.001 0.001
- link middle_bulkhead_rear: geometry collision mesh filename=package://ase389/pupper_description/Pupper_STL/Body/part3_m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 scale=0.001 0.001 0.001; visual mesh filename=package://ase389/pupper_description/Pupper_STL/Body/part3_m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 scale=0.001 0.001 0.001
- link rear_bulkhead: geometry collision mesh filename=package://ase389/pupper_description/Pupper_STL/Body/part6_r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 scale=0.001 0.001 0.001; visual mesh filename=package://ase389/pupper_description/Pupper_STL/Body/part6_r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 scale=0.001 0.001 0.001
- link top_PCB: geometry collision mesh filename=package://ase389/pupper_description/Pupper_STL/Body/PCB_Boa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 scale=0.0254 0.0254 0.0254; visual mesh filename=package://ase389/pupper_description/Pupper_STL/Body/PCB_Boa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 scale=0.0254 0.0254 0.0254
Joints:
- joint back_left_elbow_fixed_joint: child back_left_elbow -> back_left_elbow_motor
- joint back_left_elbow_joint: origin xyz=0 0 -0.032 rpy=3.14159265359 3.14159265359 0 -> xyz=-0.006 0.08 0 rpy=0 -1.5707963268 3.14159265359; parent back_left_elbow -> back_left_upper_link
- joint back_left_hip_fixed_joint: child back_left_hip -> back_left_hip_motor; origin xyz=-0.11 0.045 0.041 rpy=4.71238898039 0 1.5707963268 -> xyz=-0.110 0.045 0.041 rpy=0 1.5707963268 0
- joint back_left_hip_joint: origin xyz=0 0 0.036 rpy=0 1.5707963268 0 -> xyz=-0.147 0.045 0.041 rpy=-1.5707963268 0 0; parent back_left_hip -> bottom_PCB
- joint back_left_shoulder_fixed_joint: child back_left_shoulder -> back_left_shoulder_motor
- joint back_left_shoulder_joint: parent back_left_shoulder -> back_left_hub
- joint back_right_elbow_fixed_joint: child back_right_elbow -> back_right_elbow_motor
- joint back_right_elbow_joint: origin xyz=0 0 -0.032 rpy=3.14159265359 0 0 -> xyz=-0.006 0.08 0 rpy=0 1.5707963268 3.14159265359; parent back_right_elbow -> back_right_upper_link
- joint back_right_hip_fixed_joint: child back_right_hip -> back_right_hip_motor; origin xyz=-0.11 -0.045 0.041 rpy=4.71238898039 0 1.5707963268 -> xyz=-0.110 -0.045 0.041 rpy=4.71238898039 0 1.5707963268
- joint back_right_hip_joint: origin xyz=0 0 0.036 rpy=0 1.5707963268 0 -> xyz=-0.147 -0.045 0.041 rpy=-1.5707963268 0 0; parent back_right_hip -> bottom_PCB
- joint back_right_shoulder_fixed_joint: child back_right_shoulder -> back_right_shoulder_motor
- joint back_right_shoulder_joint: parent back_right_shoulder -> back_right_hub
- joint front_left_elbow_fixed_joint: child front_left_elbow -> front_left_elbow_motor
- joint front_left_elbow_joint: origin xyz=0 0 -0.032 rpy=3.14159265359 3.14159265359 0 -> xyz=-0.006 0.08 0 rpy=0 -1.5707963268 3.14159265359; parent front_left_elbow -> front_left_upper_link
- joint front_left_hip_fixed_joint: child front_left_hip -> front_left_hip_motor; origin xyz=0.091 0.045 0.041 rpy=4.71238898039 0 1.5707963268 -> xyz=0.091 0.045 0.041 rpy=0 1.5707963268 0
- joint front_left_hip_joint: origin xyz=0 0 0.036 rpy=0 1.5707963268 0 -> xyz=0.054 0.045 0.041 rpy=-1.5707963268 0 0; parent front_left_hip -> bottom_PCB
- joint front_left_shoulder_fixed_joint: child front_left_shoulder -> front_left_shoulder_motor
- joint front_left_shoulder_joint: parent front_left_shoulder -> front_left_hub
- joint front_right_elbow_fixed_joint: child front_right_elbow -> front_right_elbow_motor
- joint front_right_elbow_joint: origin xyz=0 0 -0.032 rpy=3.14159265359 0 0 -> xyz=-0.006 0.08 0 rpy=0 1.5707963268 3.14159265359; parent front_right_elbow -> front_right_upper_link
- joint front_right_hip_fixed_joint: child front_right_hip -> front_right_hip_motor; origin xyz=0.091 -0.045 0.041 rpy=4.71238898039 0 1.5707963268 -> xyz=0.091 -0.045 0.041 rpy=0 1.5707963268 0
- joint front_right_hip_joint: origin xyz=0 0 0.036 rpy=0 1.5707963268 0 -> xyz=0.054 -0.045 0.041 rpy=-1.5707963268 0 0; parent front_right_hip -> bottom_PCB
- joint front_right_shoulder_fixed_joint: child front_right_shoulder -> front_right_shoulder_motor
- joint front_right_shoulder_joint: parent front_right_shoulder -> front_right_hub

File: pupper_description/pupper.urdf.xacro (robot description, xacro)
@@ -272,14 +272,19 @@
     </joint>
     <xacro:leftLeg name = "front" parent = "bottom_PCB">
-        <origin xyz = "0.091 0.045 0.041" rpy = "${3*PI/2} 0 ${PI/2}"/>
+        <!-- <origin xyz = "0.091 0.045 0.041" rpy = "0 0 0"/> -->
+        <origin xyz = "0.091 0.045 0.041" rpy = "0 ${PI/2} 0"/>
+        <origin xyz = "0.054 0.045 0.041" rpy = "${-PI/2} 0 0"/>
     </xacro:leftLeg>
     <xacro:leftLeg name = "back" parent = "bottom_PCB">
-        <origin xyz = "-0.11 0.045 0.041" rpy = "${3*PI/2} 0 ${PI/2}"/>
+        <origin xyz = "-0.110 0.045 0.041" rpy = "0 ${PI/2} 0"/>
+        <origin xyz = "-0.147 0.045 0.041" rpy = "${-PI/2} 0 0"/>
     </xacro:leftLeg>
     <xacro:rightLeg name = "front" parent = "bottom_PCB">
-        <origin xyz = "0.091 -0.045 0.041" rpy = "${3*PI/2} 0 ${PI/2}"/>
+        <origin xyz = "0.091 -0.045 0.041" rpy = "0 ${PI/2} 0"/>
+        <origin xyz = "0.054 -0.045 0.041" rpy = "${-PI/2} 0 0"/>
     </xacro:rightLeg>
     <xacro:rightLeg name = "back" parent = "bottom_PCB">
-        <origin xyz = "-0.11 -0.045 0.041" rpy = "${3*PI/2} 0 ${PI/2}"/>
+        <origin xyz = "-0.110 -0.045 0.041" rpy = "${3*PI/2} 0 ${PI/2}"/>
+        <origin xyz = "-0.147 -0.045 0.041" rpy = "${-PI/2} 0 0"/>
     </xacro:rightLeg>
 </robot>

File: pupper_description/right_leg.xacro (robot description, xacro)
@@ -2,5 +2,5 @@
 <robot name = "right_leg_macro" xmlns:xacro="http://www.ros.org/wiki/xacro">
     <!-- Macro for the creation of a leg -->
-    <xacro:macro name = "rightLeg" params = "name parent *origin">
+    <xacro:macro name = "rightLeg" params = "name parent *origin *origin2">
         <!-- Create hub that connects to the motor -->
         <xacro:property name = "hubName" value = "${name}_right_hub"/>
@@ -121,5 +121,6 @@
         <xacro:motor name = "${name}_right_hip" axis = "-1 0 0" fixed_parent = "${parent}" revolute_child = "${hubName}">
             <xacro:insert_block name = "origin"/>
-            <origin xyz = "0 0 0.036" rpy = "0 ${PI/2} 0"/>
+            <xacro:insert_block name = "origin2"/>
+            <!-- <origin xyz = "0 0 0.036" rpy = "0 ${PI/2} 0"/> -->
         </xacro:motor>
         <!-- Join the Hub and the Upper Link with a motor -->
@@ -131,5 +132,6 @@
         <xacro:motor name = "${name}_right_elbow" axis = "0 0 1" fixed_parent = "${upperName}" revolute_child = "${lowerName}">
             <origin xyz = "0.023 0.082 0" rpy = "0 ${PI/2} 0"/>
-            <origin xyz = "0 0 -0.032" rpy = "${PI} 0 0"/>
+            <origin xyz = "-0.006 0.08 0" rpy = "0 ${PI/2} ${PI}"/>
+            <!-- <origin xyz = "0 0 -0.032" rpy = "${PI} 0 0"/>  -->
         </xacro:motor>
     </xacro:macro>

Commit message: Modified Gazebo sim to be more stable

File: pupper_description/left_leg.xacro (robot description, xacro)
@@ -112,4 +112,17 @@
             </xacro:if>
         </link>
+        <xacro:if value = "${full_urdf}">
+        <gazebo reference="${lowerName}">
+            <collision>
+                <surface>
+                    <contact>
+                        <ode>
+                            <min_depth>0.01</min_depth>
+                        </ode>
+                    </contact>
+                </surface>
+            </collision>
+        </gazebo>
+        </xacro:if>
         <!-- Connect foot pad to lower link -->
         <joint name = "${name}_left_foot_joint" type = "fixed">

File: pupper_description/motor.xacro (robot description, xacro)
@@ -56,5 +56,5 @@
         </gazebo>
         <gazebo reference = "${revolute_child}">
-            <self_collide>true</self_collide>
+            <self_collide>false</self_collide>
         </gazebo>
         </xacro:if>

File: pupper_description/right_leg.xacro (robot description, xacro)
@@ -112,4 +112,17 @@
             </xacro:if>
         </link>
+        <xacro:if value = "${full_urdf}">
+        <gazebo reference="${lowerName}">
+            <collision>
+                <surface>
+                    <contact>
+                        <ode>
+                            <min_depth>0.01</min_depth>
+                        </ode>
+                    </contact>
+                </surface>
+            </collision>
+        </gazebo>
+        </xacro:if>
         <!-- Connect foot pad to lower link -->
         <joint name = "${name}_right_foot_joint" type = "fixed">
