Commit message: Fixed some missing collision tags

File: pupper_description/motor.xacro (robot description, xacro)
@@ -20,5 +20,5 @@
             <collision name = "${name}_collision">
                 <geometry>
-                    <cylinder radius = "{motorRad}" length = "${motorLength}"/>
+                    <cylinder radius = "${motorRad}" length = "${motorLength}"/>
                 </geometry>
             </collision>

File: pupper_description/pupper.urdf (robot description, URDF)
Before this commit: robot pupper, 41 links, 40 joints
Links:
- link back_left_elbow: geometry collision cylinder length=0.03 radius=0.012; visual cylinder length=0.03 radius=0.012
- link back_left_shoulder_1: geometry collision cylinder length=0.03 radius=0.012; visual cylinder length=0.03 radius=0.012
- link back_left_shoulder_2: geometry collision cylinder length=0.03 radius=0.012; visual cylinder length=0.03 radius=0.012
- link back_right_elbow: geometry collision cylinder length=0.03 radius=0.012; visual cylinder length=0.03 radius=0.012
- link back_right_shoulder_1: geometry collision cylinder length=0.03 radius=0.012; visual cylinder length=0.03 radius=0.012
- link back_right_shoulder_2: geometry collision cylinder length=0.03 radius=0.012; visual cylinder length=0.03 radius=0.012
- link front_left_elbow: geometry collision cylinder length=0.03 radius=0.012; visual cylinder length=0.03 radius=0.012
- link front_left_shoulder_1: geometry collision cylinder length=0.03 radius=0.012; visual cylinder length=0.03 radius=0.012
- link front_left_shoulder_2: geometry collision cylinder length=0.03 radius=0.012; visual cylinder length=0.03 radius=0.012
- link front_right_elbow: geometry collision cylinder length=0.03 radius=0.012; visual cylinder length=0.03 radius=0.012
- link front_right_shoulder_1: geometry collision cylinder length=0.03 radius=0.012; visual cylinder length=0.03 radius=0.012
- link front_right_shoulder_2: geometry collision cylinder length=0.03 radius=0.012; visual cylinder length=0.03 radius=0.012
- link middle_bulkhead_front: geometry collision mesh filename=package://ase389/pupper_description/Pupper_STL/Body/part2_m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 scale=0.001 0.001 0.001; visual mesh filename=package://ase389/pupper_description/Pupper_STL/Body/part2_m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 scale=0.001 0.001 0.001
- link middle_bulkhead_rear: geometry collision mesh filename=package://ase389/pupper_description/Pupper_STL/Body/part3_m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 scale=0.001 0.001 0.001; visual mesh filename=package://ase389/pupper_description/Pupper_STL/Body/part3_m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 scale=0.001 0.001 0.001

File: pupper_description/pupper.urdf.xacro (robot description, xacro)
@@ -95,5 +95,5 @@
         <collision name = "middle_bulkhead_front_collision">
             <geometry>
-                <mesh filename = "${CollisionPath}/Body/part2_middlebulkhead1_simplified.dae" scale = "{meshScale_mm}"/>
+                <mesh filename = "${CollisionPath}/Body/part2_middlebulkhead1_simplified.dae" scale = "${meshScale_mm}"/>
             </geometry>
         </collision>
@@ -119,5 +119,5 @@
         <collision name = "middle_bulkhead_rear_collision">
             <geometry>
-                <mesh filename = "${CollisionPath}/Body/part3_middlebulkhead2_simplified.dae" scale = "{meshScale_mm}"/>
+                <mesh filename = "${CollisionPath}/Body/part3_middlebulkhead2_simplified.dae" scale = "${meshScale_mm}"/>
             </geometry>
         </collision>

Commit message: Reduced damping

File: pupper_description/motor.xacro (robot description, xacro)
@@ -38,5 +38,5 @@
             <xacro:insert_block name = "revolute_origin"/>
             <limit upper = "1e10" lower = "-1e10" effort = "1e6" velocity = "1e6"/>
-            <dynamics damping = "0.3" friction = "0.3"/>
+            <dynamics damping = "0.2" friction = "0.3"/>
             <axis xyz = "${axis}"/>
         </joint>

Commit message: Measurements

File: pupper_description/motor.xacro (robot description, xacro)
@@ -4,5 +4,5 @@
         <xacro:property name = "motorRad"    value = "0.012"/>
         <xacro:property name = "motorLength" value = "0.03"/>
-        <xacro:property name = "motorMass"   value = "0.120"/> <!-- kg -->
+        <xacro:property name = "motorMass"   value = "0.09"/> <!-- kg -->
         <!-- Create the motor -->
         <link name = "${name}_motor">
@@ -56,5 +56,5 @@
         </gazebo>
         <gazebo reference = "${revolute_child}">
-            <self_collide>false</self_collide>
+            <self_collide>true</self_collide>
         </gazebo>
         </xacro:if>

Commit message: Updated model with new mass measurements

File: pupper_description/motor.xacro (robot description, xacro)
@@ -56,5 +56,5 @@
         </gazebo>
         <gazebo reference = "${revolute_child}">
-            <self_collide>true</self_collide>
+            <self_collide>false</self_collide>
         </gazebo>
         </xacro:if>

File: pupper_description/pupper.urdf.xacro (robot description, xacro)
@@ -29,5 +29,5 @@
     <!-- Inertia of a hemisphere via Wikipedia -->
     <xacro:macro name = "footInertia">
-        <xacro:property name = "foot_mass" value = "0.01"/>
+        <xacro:property name = "foot_mass" value = "0.003"/>
         <xacro:property name = "foot_radius" value = "0.0095"/>
         <xacro:property name = "i__" value = "${2/5 * foot_mass * foot_radius**2}"/>
